Commit message: Problem with the wrist and ROS fix

File: qibullet/robot_data/pepper_1.7/pepper_rGripper.urdf (robot description, URDF)
Before this commit: robot RGripper, 18 links, 17 joints
Links:
- link r_wrist: geometry collision mesh filename=meshes/RWristYaw_vahcd.obj scale=0.1 0.1 0.1; visual mesh filename=meshes/RWristYaw.obj scale=0.1 0.1 0.1
