Commit message: update point grasp

File: grasp_point/data/robot_data/pepper_1.7/pepper_LGripper.urdf (robot description, URDF)
Before this commit: robot LGripper, 18 links, 17 joints
Links:
- added link l_eef, mass 2e-03
- link LFinger11_link: geometry collision mesh filename=meshes/LFinger11.obj scale=0.1 0.1 0.1; visual mesh filename=meshes/LFinger11.obj scale=0.1 0.1 0.1
- link LFinger12_link: geometry collision mesh filename=meshes/LFinger12.obj scale=0.1 0.1 0.1; visual mesh filename=meshes/LFinger12.obj scale=0.1 0.1 0.1
- link LFinger13_link: geometry collision mesh filename=meshes/LFinger13.obj scale=0.1 0.1 0.1; visual mesh filename=meshes/LFinger13.obj scale=0.1 0.1 0.1
- link LFinger21_link: geometry collision mesh filename=meshes/LFinger21.obj scale=0.1 0.1 0.1; visual mesh filename=meshes/LFinger21.obj scale=0.1 0.1 0.1
- link LFinger22_link: geometry collision mesh filename=meshes/LFinger22.obj scale=0.1 0.1 0.1; visual mesh filename=meshes/LFinger22.obj scale=0.1 0.1 0.1
- link LFinger23_link: geometry collision mesh filename=meshes/LFinger23.obj scale=0.1 0.1 0.1; visual mesh filename=meshes/LFinger23.obj scale=0.1 0.1 0.1
- link LFinger31_link: geometry collision mesh filename=meshes/LFinger31.obj scale=0.1 0.1 0.1; visual mesh filename=meshes/LFinger31.obj scale=0.1 0.1 0.1
- link LFinger32_link: geometry collision mesh filename=meshes/LFinger32.obj scale=0.1 0.1 0.1; visual mesh filename=meshes/LFinger32.obj scale=0.1 0.1 0.1
- link LFinger33_link: geometry collision mesh filename=meshes/LFinger33.obj scale=0.1 0.1 0.1; visual mesh filename=meshes/LFinger33.obj scale=0.1 0.1 0.1
- link LFinger41_link: geometry collision mesh filename=meshes/LFinger41.obj scale=0.1 0.1 0.1; visual mesh filename=meshes/LFinger41.obj scale=0.1 0.1 0.1
- link LFinger42_link: geometry collision mesh filename=meshes/LFinger42.obj scale=0.1 0.1 0.1; visual mesh filename=meshes/LFinger42.obj scale=0.1 0.1 0.1
- link LFinger43_link: geometry collision mesh filename=meshes/LFinger43.obj scale=0.1 0.1 0.1; visual mesh filename=meshes/LFinger43.obj scale=0.1 0.1 0.1
- link LThumb1_link: geometry collision mesh filename=meshes/LThumb1.obj scale=0.1 0.1 0.1; visual mesh filename=meshes/LThumb1.obj scale=0.1 0.1 0.1
- link LThumb2_link: geometry collision mesh filename=meshes/LThumb2.obj scale=0.1 0.1 0.1; visual mesh filename=meshes/LThumb2.obj scale=0.1 0.1 0.1
Joints:
- removed joint LHand/Touch/Back_sensol_fixedjoint
- added joint LGripperEef: type fixed, parent l_gripper, child l_eef, origin xyz=0.020 0 -0.005 rpy=3.14 -0.785 0, axis 0 0 0, limit lower=0.02 upper=0.98 effort=0.144 velocity=12.56
- added joint LHand/Touch/Back_sensor_fixedjoint: type fixed, parent l_wrist, child LHandTouchBack_frame, origin xyz=0.0523 0 0.0304 rpy=1.5708 -1.5708 -3.14159, axis 0 0 0
- joint LFinger11: origin xyz=0.0821 0.0268 0.004 rpy=1.39757 1.04064 0.0334335 -> xyz=0.0821 -0.0268 0.004 rpy=1.74402 1.04064 -0.0334335
- joint LFinger21: origin xyz=0.0873 0.0073 0.006 rpy=1.5708 1.0472 0.061086 -> xyz=0.0873 -0.0073 0.006 rpy=1.5708 1.0472 -0.061086
- joint LFinger31: origin xyz=0.0833 -0.0123 0.004 rpy=1.67523 1.04483 0.029316 -> xyz=0.0833 0.0123 0.004 rpy=1.46636 1.04483 -0.029314
- joint LFinger41: origin xyz=0.074 -0.0309 0 rpy=1.74402 1.04064 -0.0683394 -> xyz=0.074 0.0309 0 rpy=1.39757 1.04064 0.0683394
- joint LHand: origin xyz=0.025 0 0 rpy=0.6 0 0 -> xyz=0.025 0 0 rpy=0 0 0

File: grasp_point/data/robot_data/pepper_1.7/pepper_RGripper.urdf (robot description, URDF)
Before this commit: robot RGripper, 18 links, 17 joints
Links:
- added link r_eef, mass 2e-03
- link RFinger11_link: geometry collision mesh filename=meshes/RFinger11.obj scale=0.1 0.1 0.1; visual mesh filename=meshes/RFinger11.obj scale=0.1 0.1 0.1
- link RFinger12_link: geometry collision mesh filename=meshes/RFinger12.obj scale=0.1 0.1 0.1; visual mesh filename=meshes/RFinger12.obj scale=0.1 0.1 0.1
- link RFinger13_link: geometry collision mesh filename=meshes/RFinger13.obj scale=0.1 0.1 0.1; visual mesh filename=meshes/RFinger13.obj scale=0.1 0.1 0.1
- link RFinger21_link: geometry collision mesh filename=meshes/RFinger21.obj scale=0.1 0.1 0.1; visual mesh filename=meshes/RFinger21.obj scale=0.1 0.1 0.1
- link RFinger22_link: geometry collision mesh filename=meshes/RFinger22.obj scale=0.1 0.1 0.1; visual mesh filename=meshes/RFinger22.obj scale=0.1 0.1 0.1
- link RFinger23_link: geometry collision mesh filename=meshes/RFinger23.obj scale=0.1 0.1 0.1; visual mesh filename=meshes/RFinger23.obj scale=0.1 0.1 0.1
- link RFinger31_link: geometry collision mesh filename=meshes/RFinger31.obj scale=0.1 0.1 0.1; visual mesh filename=meshes/RFinger31.obj scale=0.1 0.1 0.1
- link RFinger32_link: geometry collision mesh filename=meshes/RFinger32.obj scale=0.1 0.1 0.1; visual mesh filename=meshes/RFinger32.obj scale=0.1 0.1 0.1
- link RFinger33_link: geometry collision mesh filename=meshes/RFinger33.obj scale=0.1 0.1 0.1; visual mesh filename=meshes/RFinger33.obj scale=0.1 0.1 0.1
- link RFinger41_link: geometry collision mesh filename=meshes/RFinger41.obj scale=0.1 0.1 0.1; visual mesh filename=meshes/RFinger41.obj scale=0.1 0.1 0.1
- link RFinger42_link: geometry collision mesh filename=meshes/RFinger42.obj scale=0.1 0.1 0.1; visual mesh filename=meshes/RFinger42.obj scale=0.1 0.1 0.1
- link RFinger43_link: geometry collision mesh filename=meshes/RFinger43.obj scale=0.1 0.1 0.1; visual mesh filename=meshes/RFinger43.obj scale=0.1 0.1 0.1
- link RThumb1_link: geometry collision mesh filename=meshes/RThumb1.obj scale=0.1 0.1 0.1; visual mesh filename=meshes/RThumb1.obj scale=0.1 0.1 0.1
- link RThumb2_link: geometry collision mesh filename=meshes/RThumb2.obj scale=0.1 0.1 0.1; visual mesh filename=meshes/RThumb2.obj scale=0.1 0.1 0.1
Joints:
- added joint RGripperEef: type fixed, parent r_gripper, child r_eef, origin xyz=0.020 0 -0.005 rpy=3.14 -0.785 0, axis 0 0 0, limit lower=0.02 upper=0.98 effort=0.144 velocity=12.56
- joint RHand: origin xyz=0.025 0 0 rpy=0.6 0 0 -> xyz=0.025 0 0 rpy=0 0 0
